Commit message: Add files via upload

File: omni_robot_description/urdf/omni_robot.xacro (robot description, xacro)
@@ -6,7 +6,7 @@
 <link name="base_link">
   <inertial>
-    <origin xyz="-0.0003866035215641167 1.8970697824213494e-17 0.014105491397793652" rpy="0 0 0"/>
+    <origin xyz="-0.00039055834309408623 1.8970697824213494e-17 0.013449503145948333" rpy="0 0 0"/>
     <mass value="7.526906469202046"/>
-    <inertia ixx="0.018693" iyy="0.018693" izz="0.035927" ixy="0.0" iyz="0.0" ixz="3e-06"/>
+    <inertia ixx="0.018693" iyy="0.018693" izz="0.035927" ixy="-0.0" iyz="-0.0" ixz="3e-06"/>
   </inertial>
   <visual>
@@ -24,12 +24,72 @@
   </collision>
 </link>
+<link name="rim_1_1">
+  <inertial>
+    <origin xyz="0.00899995139183217 3.200222004718161e-14 -3.8621820508226434e-07" rpy="0 0 0"/>
+    <mass value="0.14023608587607866"/>
+    <inertia ixx="5e-05" iyy="3e-05" izz="3e-05" ixy="-0.0" iyz="-0.0" ixz="-0.0"/>
+  </inertial>
+  <visual>
+    <origin xyz="0.130374 0.0 -0.012426" rpy="0 0 0"/>
+    <geometry>
+      <mesh filename="file://$(find omni_robot_description)/meshes/rim_1_1.stl" scale="0.001 0.001 0.001"/>
+    </geometry>
+    <material name="silver"/>
+  </visual>
+  <collision>
+    <origin xyz="0.130374 0.0 -0.012426" rpy="0 0 0"/>
+    <geometry>
+      <mesh filename="file://$(find omni_robot_description)/meshes/rim_1_1.stl" scale="0.001 0.001 0.001"/>
+    </geometry>
+  </collision>
+</link>
+<link name="rim_2_1">
+  <inertial>
+    <origin xyz="-4.860822816189726e-08 0.008999999999999966 -3.8621817657555346e-07" rpy="0 0 0"/>
+    <mass value="0.1402360858760785"/>
+    <inertia ixx="3e-05" iyy="5e-05" izz="3e-05" ixy="0.0" iyz="-0.0" ixz="0.0"/>
+  </inertial>
+  <visual>
+    <origin xyz="0.000374 0.13 -0.012426" rpy="0 0 0"/>
+    <geometry>
+      <mesh filename="file://$(find omni_robot_description)/meshes/rim_2_1.stl" scale="0.001 0.001 0.001"/>
+    </geometry>
+    <material name="silver"/>
+  </visual>
+  <collision>
+    <origin xyz="0.000374 0.13 -0.012426" rpy="0 0 0"/>
+    <geometry>
+      <mesh filename="file://$(find omni_robot_description)/meshes/rim_2_1.stl" scale="0.001 0.001 0.001"/>
+    </geometry>
+  </collision>
+</link>
+<link name="rim_3_1">
+  <inertial>
+    <origin xyz="-0.009000048608167707 3.2057903750967407e-14 -3.8621820497818093e-07" rpy="0 0 0"/>
+    <mass value="0.14023608587607866"/>
+    <inertia ixx="5e-05" iyy="3e-05" izz="3e-05" ixy="-0.0" iyz="-0.0" ixz="0.0"/>
+  </inertial>
+  <visual>
+    <origin xyz="-0.129626 0.0 -0.012426" rpy="0 0 0"/>
+    <geometry>
+      <mesh filename="file://$(find omni_robot_description)/meshes/rim_3_1.stl" scale="0.001 0.001 0.001"/>
+    </geometry>
+    <material name="silver"/>
+  </visual>
+  <collision>
+    <origin xyz="-0.129626 0.0 -0.012426" rpy="0 0 0"/>
+    <geometry>
+      <mesh filename="file://$(find omni_robot_description)/meshes/rim_3_1.stl" scale="0.001 0.001 0.001"/>
+    </geometry>
+  </collision>
+</link>
 <link name="rim_4_1">
   <inertial>
-    <origin xyz="-1.1325643013986204e-07 -0.009000000000000077 3.8076191856070696e-07" rpy="0 0 0"/>
+    <origin xyz="-4.860822806258434e-08 -0.009000000000000077 -3.8621817657555346e-07" rpy="0 0 0"/>
     <mass value="0.14023608587607855"/>
-    <inertia ixx="3e-05" iyy="5e-05" izz="3e-05" ixy="-0.0" iyz="0.0" ixz="0.0"/>
-  </inertial>
-  <visual>
-    <origin xyz="0.000403 -0.13 -0.015129" rpy="0 0 0"/>
+    <inertia ixx="3e-05" iyy="5e-05" izz="3e-05" ixy="0.0" iyz="-0.0" ixz="0.0"/>
+  </inertial>
+  <visual>
+    <origin xyz="0.000374 -0.13 -0.012426" rpy="0 0 0"/>
     <geometry>
       <mesh filename="file://$(find omni_robot_description)/meshes/rim_4_1.stl" scale="0.001 0.001 0.001"/>
@@ -38,5 +98,5 @@
   </visual>
   <collision>
-    <origin xyz="0.000403 -0.13 -0.015129" rpy="0 0 0"/>
+    <origin xyz="0.000374 -0.13 -0.012426" rpy="0 0 0"/>
     <geometry>
       <mesh filename="file://$(find omni_robot_description)/meshes/rim_4_1.stl" scale="0.001 0.001 0.001"/>
@@ -44,61 +104,81 @@
   </collision>
 </link>
-<link name="rim_1_1">
-  <inertial>
-    <origin xyz="-0.009000113256490583 3.200222004718161e-14 3.8076194701537613e-07" rpy="0 0 0"/>
-    <mass value="0.14023608587607866"/>
-    <inertia ixx="5e-05" iyy="3e-05" izz="3e-05" ixy="0.0" iyz="0.0" ixz="-0.0"/>
-  </inertial>
-  <visual>
-    <origin xyz="-0.129597 0.0 -0.015129" rpy="0 0 0"/>
-    <geometry>
-      <mesh filename="file://$(find omni_robot_description)/meshes/rim_1_1.stl" scale="0.001 0.001 0.001"/>
-    </geometry>
-    <material name="silver"/>
-  </visual>
-  <collision>
-    <origin xyz="-0.129597 0.0 -0.015129" rpy="0 0 0"/>
-    <geometry>
-      <mesh filename="file://$(find omni_robot_description)/meshes/rim_1_1.stl" scale="0.001 0.001 0.001"/>
-    </geometry>
-  </collision>
-</link>
-<link name="rim_2_1">
-  <inertial>
-    <origin xyz="-1.1325643004054912e-07 0.008999999999999966 3.8076191856070696e-07" rpy="0 0 0"/>
-    <mass value="0.1402360858760785"/>
-    <inertia ixx="3e-05" iyy="5e-05" izz="3e-05" ixy="-0.0" iyz="0.0" ixz="0.0"/>
-  </inertial>
-  <visual>
-    <origin xyz="0.000403 0.13 -0.015129" rpy="0 0 0"/>
-    <geometry>
-      <mesh filename="file://$(find omni_robot_description)/meshes/rim_2_1.stl" scale="0.001 0.001 0.001"/>
-    </geometry>
-    <material name="silver"/>
-  </visual>
-  <collision>
-    <origin xyz="0.000403 0.13 -0.015129" rpy="0 0 0"/>
-    <geometry>
-      <mesh filename="file://$(find omni_robot_description)/meshes/rim_2_1.stl" scale="0.001 0.001 0.001"/>
-    </geometry>
-  </collision>
-</link>
-<link name="rim_3_1">
-  <inertial>
-    <origin xyz="0.008999886743509697 3.2057903750967407e-14 3.8076194701537613e-07" rpy="0 0 0"/>
-    <mass value="0.14023608587607866"/>
-    <inertia ixx="5e-05" iyy="3e-05" izz="3e-05" ixy="0.0" iyz="0.0" ixz="-0.0"/>
-  </inertial>
-  <visual>
-    <origin xyz="0.130403 0.0 -0.015129" rpy="0 0 0"/>
-    <geometry>
-      <mesh filename="file://$(find omni_robot_description)/meshes/rim_3_1.stl" scale="0.001 0.001 0.001"/>
-    </geometry>
-    <material name="silver"/>
-  </visual>
-  <collision>
-    <origin xyz="0.130403 0.0 -0.015129" rpy="0 0 0"/>
-    <geometry>
-      <mesh filename="file://$(find omni_robot_description)/meshes/rim_3_1.stl" scale="0.001 0.001 0.001"/>
+<link name="roller_1_2_1">
+  <inertial>
+    <origin xyz="-4.8608167907415734e-08 -0.007152434060027909 0.005157276950545811" rpy="0 0 0"/>
+    <mass value="0.017098974596301414"/>
+    <inertia ixx="1e-06" iyy="0.0" izz="1e-06" ixy="0.0" iyz="0.0" ixz="-0.0"/>
+  </inertial>
+  <visual>
+    <origin xyz="0.128124 -0.020392 -0.024892" rpy="0 0 0"/>
+    <geometry>
+      <mesh filename="file://$(find omni_robot_description)/meshes/roller_1_2_1.stl" scale="0.001 0.001 0.001"/>
+    </geometry>
+    <material name="silver"/>
+  </visual>
+  <collision>
+    <origin xyz="0.128124 -0.020392 -0.024892" rpy="0 0 0"/>
+    <geometry>
+      <mesh filename="file://$(find omni_robot_description)/meshes/roller_1_2_1.stl" scale="0.001 0.001 0.001"/>
+    </geometry>
+  </collision>
+</link>
+<link name="roller_1_1_1">
+  <inertial>
+    <origin xyz="-4.860816793517131e-08 0.002695350571172799 0.00839604974399046" rpy="0 0 0"/>
+    <mass value="0.017098974596301386"/>
+    <inertia ixx="1e-06" iyy="1e-06" izz="0.0" ixy="-0.0" iyz="-0.0" ixz="0.0"/>
+  </inertial>
+  <visual>
+    <origin xyz="0.128124 -0.018157 0.003116" rpy="0 0 0"/>
+    <geometry>
+      <mesh filename="file://$(find omni_robot_description)/meshes/roller_1_1_1.stl" scale="0.001 0.001 0.001"/>
+    </geometry>
+    <material name="silver"/>
+  </visual>
+  <collision>
+    <origin xyz="0.128124 -0.018157 0.003116" rpy="0 0 0"/>
+    <geometry>
+      <mesh filename="file://$(find omni_robot_description)/meshes/roller_1_1_1.stl" scale="0.001 0.001 0.001"/>
+    </geometry>
+  </collision>
+</link>
+<link name="roller_1_5_1">
+  <inertial>
+    <origin xyz="-4.860816793517131e-08 0.008817895458340549 3.174916897563142e-05" rpy="0 0 0"/>
+    <mass value="0.017098974596301345"/>
+    <inertia ixx="1e-06" iyy="0.0" izz="1e-06" ixy="0.0" iyz="-0.0" ixz="0.0"/>
+  </inertial>
+  <visual>
+    <origin xyz="0.128124 0.00917 0.009646" rpy="0 0 0"/>
+    <geometry>
+      <mesh filename="file://$(find omni_robot_description)/meshes/roller_1_5_1.stl" scale="0.001 0.001 0.001"/>
+    </geometry>
+    <material name="silver"/>
+  </visual>
+  <collision>
+    <origin xyz="0.128124 0.00917 0.009646" rpy="0 0 0"/>
+    <geometry>
+      <mesh filename="file://$(find omni_robot_description)/meshes/roller_1_5_1.stl" scale="0.001 0.001 0.001"/>
+    </geometry>
+  </collision>
+</link>
+<link name="roller_1_3_1">
+  <inertial>
+    <origin xyz="-4.860816787966016e-08 0.0027550368544883505 -0.008377207618485365" rpy="0 0 0"/>
+    <mass value="0.01709897459630136"/>
+    <inertia ixx="1e-06" iyy="1e-06" izz="0.0" ixy="-0.0" iyz="0.0" ixz="-0.0"/>
+  </inertial>
+  <visual>
+    <origin xyz="0.128124 0.023825 -0.014327" rpy="0 0 0"/>
+    <geometry>
+      <mesh filename="file://$(find omni_robot_description)/meshes/roller_1_3_1.stl" scale="0.001 0.001 0.001"/>
+    </geometry>
+    <material name="silver"/>
+  </visual>
+  <collision>
+    <origin xyz="0.128124 0.023825 -0.014327" rpy="0 0 0"/>
+    <geometry>
+      <mesh filename="file://$(find omni_robot_description)/meshes/roller_1_3_1.stl" scale="0.001 0.001 0.001"/>
     </geometry>
   </collision>
@@ -106,10 +186,10 @@
 <link name="roller_1_4_1">
   <inertial>
-    <origin xyz="-1.1325649029725326e-07 -0.007115848823974879 0.005208793879491304" rpy="0 0 0"/>
+    <origin xyz="-4.860816810170476e-08 -0.0071158488239748425 -0.005208799335749234" rpy="0 0 0"/>
     <mass value="0.017098974596301365"/>
-    <inertia ixx="1e-06" iyy="0.0" izz="1e-06" ixy="-0.0" iyz="0.0" ixz="-0.0"/>
-  </inertial>
-  <visual>
-    <origin xyz="-0.127347 0.005554 0.008117" rpy="0 0 0"/>
+    <inertia ixx="1e-06" iyy="0.0" izz="1e-06" ixy="0.0" iyz="-0.0" ixz="-0.0"/>
+  </inertial>
+  <visual>
+    <origin xyz="0.128124 0.005554 -0.035672" rpy="0 0 0"/>
     <geometry>
       <mesh filename="file://$(find omni_robot_description)/meshes/roller_1_4_1.stl" scale="0.001 0.001 0.001"/>
@@ -118,5 +198,5 @@
   </visual>
   <collision>
-    <origin xyz="-0.127347 0.005554 0.008117" rpy="0 0 0"/>
+    <origin xyz="0.128124 0.005554 -0.035672" rpy="0 0 0"/>
     <geometry>
       <mesh filename="file://$(find omni_robot_description)/meshes/roller_1_4_1.stl" scale="0.001 0.001 0.001"/>
@@ -124,312 +204,692 @@
   </collision>
 </link>
-<link name="roller_1_2_1">
-  <inertial>
-    <origin xyz="-1.1325649040827557e-07 0.007134541942991805 0.005183111093174693" rpy="0 0 0"/>
-    <mass value="0.01709897459630134"/>
+<link name="roller_1_9_1">
+  <inertial>
+    <origin xyz="-4.8608168018438036e-08 0.007097166613708081 0.005234847529153874" rpy="0 0 0"/>
+    <mass value="0.017098974596301372"/>
+    <inertia ixx="1e-06" iyy="0.0" izz="1e-06" ixy="-0.0" iyz="-0.0" ixz="0.0"/>
+  </inertial>
+  <visual>
+    <origin xyz="0.114624 -0.005568 0.010811" rpy="0 0 0"/>
+    <geometry>
+      <mesh filename="file://$(find omni_robot_description)/meshes/roller_1_9_1.stl" scale="0.001 0.001 0.001"/>
+    </geometry>
+    <material name="silver"/>
+  </visual>
+  <collision>
+    <origin xyz="0.114624 -0.005568 0.010811" rpy="0 0 0"/>
+    <geometry>
+      <mesh filename="file://$(find omni_robot_description)/meshes/roller_1_9_1.stl" scale="0.001 0.001 0.001"/>
+    </geometry>
+  </collision>
+</link>
+<link name="roller_1_7_1">
+  <inertial>
+    <origin xyz="-4.860816785190458e-08 0.007171054620771836 -0.005131527156925909" rpy="0 0 0"/>
+    <mass value="0.017098974596301407"/>
+    <inertia ixx="1e-06" iyy="0.0" izz="1e-06" ixy="0.0" iyz="0.0" ixz="-0.0"/>
+  </inertial>
+  <visual>
+    <origin xyz="0.114624 0.020378 5.1e-05" rpy="0 0 0"/>
+    <geometry>
+      <mesh filename="file://$(find omni_robot_description)/meshes/roller_1_7_1.stl" scale="0.001 0.001 0.001"/>
+    </geometry>
+    <material name="silver"/>
+  </visual>
+  <collision>
+    <origin xyz="0.114624 0.020378 5.1e-05" rpy="0 0 0"/>
+    <geometry>
+      <mesh filename="file://$(find omni_robot_description)/meshes/roller_1_7_1.stl" scale="0.001 0.001 0.001"/>
+    </geometry>
+  </collision>
+</link>
+<link name="roller_1_6_1">
+  <inertial>
+    <origin xyz="-4.86081679490491e-08 -0.0026645077456347727 -0.00840604954430816" rpy="0 0 0"/>
+    <mass value="0.017098974596301393"/>
+    <inertia ixx="1e-06" iyy="1e-06" izz="0.0" ixy="0.0" iyz="-0.0" ixz="-0.0"/>
+  </inertial>
+  <visual>
+    <origin xyz="0.114624 0.018163 -0.027951" rpy="0 0 0"/>
+    <geometry>
+      <mesh filename="file://$(find omni_robot_description)/meshes/roller_1_6_1.stl" scale="0.001 0.001 0.001"/>
+    </geometry>
+    <material name="silver"/>
+  </visual>
+  <collision>
+    <origin xyz="0.114624 0.018163 -0.027951" rpy="0 0 0"/>
+    <geometry>
+      <mesh filename="file://$(find omni_robot_description)/meshes/roller_1_6_1.stl" scale="0.001 0.001 0.001"/>
+    </geometry>
+  </collision>
+</link>
+<link name="roller_1_10_1">
+  <inertial>
+    <origin xyz="-4.860816775476007e-08 -0.008818162308526037 -6.325323757874063e-05" rpy="0 0 0"/>
+    <mass value="0.017098974596301414"/>
     <inertia ixx="1e-06" iyy="0.0" izz="1e-06" ixy="0.0" iyz="-0.0" ixz="0.0"/>
   </inertial>
   <visual>
-    <origin xyz="-0.127347 -0.005401 0.008146" rpy="0 0 0"/>
-    <geometry>
-      <mesh filename="file://$(find omni_robot_description)/meshes/roller_1_2_1.stl" scale="0.001 0.001 0.001"/>
-    </geometry>
-    <material name="silver"/>
-  </visual>
-  <collision>
-    <origin xyz="-0.127347 -0.005401 0.008146" rpy="0 0 0"/>
-    <geometry>
-      <mesh filename="file://$(find omni_robot_description)/meshes/roller_1_2_1.stl" scale="0.001 0.001 0.001"/>
-    </geometry>
-  </collision>
-</link>
-<link name="roller_1_1_1">
-  <inertial>
-    <origin xyz="-1.1325649035276442e-07 0.0026953505711728963 -0.00839605520024855" rpy="0 0 0"/>
-    <mass value="0.01709897459630134"/>
-    <inertia ixx="1e-06" iyy="1e-06" izz="0.0" ixy="0.0" iyz="0.0" ixz="0.0"/>
-  </inertial>
-  <visual>
-    <origin xyz="-0.127347 -0.018157 -0.030671" rpy="0 0 0"/>
-    <geometry>
-      <mesh filename="file://$(find omni_robot_description)/meshes/roller_1_1_1.stl" scale="0.001 0.001 0.001"/>
-    </geometry>
-    <material name="silver"/>
-  </visual>
-  <collision>
-    <origin xyz="-0.127347 -0.018157 -0.030671" rpy="0 0 0"/>
-    <geometry>
-      <mesh filename="file://$(find omni_robot_description)/meshes/roller_1_1_1.stl" scale="0.001 0.001 0.001"/>
-    </geometry>
-  </collision>
-</link>
-<link name="roller_1_5_1">
-  <inertial>
-    <origin xyz="-1.1325649046378672e-07 0.00881789545834062 -3.175462523376249e-05" rpy="0 0 0"/>
-    <mass value="0.01709897459630137"/>
-    <inertia ixx="1e-06" iyy="0.0" izz="1e-06" ixy="-0.0" iyz="0.0" ixz="0.0"/>
-  </inertial>
-  <visual>
-    <origin xyz="-0.127347 0.00917 -0.037201" rpy="0 0 0"/>
-    <geometry>
-      <mesh filename="file://$(find omni_robot_description)/meshes/roller_1_5_1.stl" scale="0.001 0.001 0.001"/>
-    </geometry>
-    <material name="silver"/>
-  </visual>
-  <collision>
-    <origin xyz="-0.127347 0.00917 -0.037201" rpy="0 0 0"/>
-    <geometry>
-      <mesh filename="file://$(find omni_robot_description)/meshes/roller_1_5_1.stl" scale="0.001 0.001 0.001"/>
-    </geometry>
-  </collision>
-</link>
-<link name="roller_1_3_1">
-  <inertial>
-    <origin xyz="-1.132564904915423e-07 0.0027550368544883505 0.00837720216222736" rpy="0 0 0"/>
+    <origin xyz="0.114624 -0.009153 -0.034497" rpy="0 0 0"/>
+    <geometry>
+      <mesh filename="file://$(find omni_robot_description)/meshes/roller_1_10_1.stl" scale="0.001 0.001 0.001"/>
+    </geometry>
+    <material name="silver"/>
+  </visual>
+  <collision>
+    <origin xyz="0.114624 -0.009153 -0.034497" rpy="0 0 0"/>
+    <geometry>
+      <mesh filename="file://$(find omni_robot_description)/meshes/roller_1_10_1.stl" scale="0.001 0.001 0.001"/>
+    </geometry>
+  </collision>
+</link>
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